Commit message: feat(add the imupreintegration): lio_sam

File: sim_env/husky/husky_description/urdf/husky.urdf.xacro (robot description, xacro)
@@ -124,10 +124,10 @@
     <origin xyz="${wheelbase/2} ${-track/2} ${wheel_vertical_offset}" rpy="0 0 0" />
   </xacro:husky_wheel>
-  <xacro:husky_wheel wheel_prefix="rear_left">
+  <xacro:drive_husky_wheel wheel_prefix="rear_left">
     <origin xyz="${-wheelbase/2} ${track/2} ${wheel_vertical_offset}" rpy="0 0 0" />
-  </xacro:husky_wheel>
-  <xacro:husky_wheel wheel_prefix="rear_right">
+  </xacro:drive_husky_wheel>
+  <xacro:drive_husky_wheel wheel_prefix="rear_right">
     <origin xyz="${-wheelbase/2} ${-track/2} ${wheel_vertical_offset}" rpy="0 0 0" />
-  </xacro:husky_wheel>
+  </xacro:drive_husky_wheel>
   <xacro:husky_decorate />
   <!--
@@ -181,9 +181,9 @@
     <plugin name="imu_controller" filename="libhector_gazebo_ros_imu.so">
       <robotNamespace>$(arg robot_namespace)</robotNamespace>
-      <updateRate>50.0</updateRate>
+      <updateRate>100.0</updateRate>
       <bodyName>base_link</bodyName>
       <topicName>imu/data</topicName>
-      <accelDrift>0.005 0.005 0.005</accelDrift>
-      <accelGaussianNoise>0.05 0.05 0.05</accelGaussianNoise>
+      <accelDrift>0.0 0.0 0.0</accelDrift>
+      <accelGaussianNoise>0.0 0.0 0.0</accelGaussianNoise>
       <!-- <rateDrift>0.005 0.005 0.005 </rateDrift> -->
       <!-- <rateGaussianNoise>0.005 0.005 0.005 </rateGaussianNoise> -->
@@ -196,5 +196,5 @@
     <plugin name="p3d_base_controller" filename="libgazebo_ros_p3d.so">
       <alwaysOn>true</alwaysOn>
-      <updateRate>20.0</updateRate>
+      <updateRate>50.0</updateRate>
       <bodyName>base_link</bodyName>
       <topicName>ground_truth/state</topicName>

File: sim_env/husky/husky_description/urdf/wheel.urdf.xacro (robot description, xacro)
@@ -22,5 +22,5 @@
 -->
 <robot xmlns:xacro="http://ros.org/wiki/xacro" name="husky_wheel">
-	<xacro:macro name="husky_wheel" params="wheel_prefix *joint_pose">
+	<xacro:macro name="drive_husky_wheel" params="wheel_prefix *joint_pose">
 		<link name="${wheel_prefix}_wheel_link">
 			<inertial>
@@ -43,6 +43,6 @@
 		</link>
 		<gazebo reference="${wheel_prefix}_wheel_link">
-			<mu1 value="1.0"/>
-			<mu2 value="1.0"/>
+			<mu1 value="1"/>
+			<mu2 value="1"/>
 			<kp value="10000000.0" />
 			<kd value="1.0" />
@@ -65,3 +65,43 @@
 		</transmission>
 	</xacro:macro>
+		<xacro:macro name="husky_wheel" params="wheel_prefix *joint_pose">
+		<link name="${wheel_prefix}_wheel_link">
+			<inertial>
+				<mass value="2.637" />
+				<origin xyz="0 0 0" />
+				<inertia  ixx="0.02467" ixy="0" ixz="0" iyy="0.04411" iyz="0" izz="0.02467" />
+			</inertial>
+			<visual>
+				<origin xyz="0 0 0" rpy="0 0 0" />
+				<geometry>
+					<mesh filename="package://husky_description/meshes/wheel.dae" />
+				</geometry>
+			</visual>
+			<collision>
+				<origin xyz="0 0 0" rpy="${M_PI/2} 0 0" />
+				<geometry>
+					<cylinder length="${wheel_length}" radius="${wheel_radius}" />
+				</geometry>
+			</collision>
+		</link>
+		<gazebo reference="${wheel_prefix}_wheel_link">
+			<mu1 value="0"/>
+			<mu2 value="0"/>
+		</gazebo>
+		<joint name="${wheel_prefix}_wheel" type="continuous">
+			<parent link="base_link"/>
+			<child link="${wheel_prefix}_wheel_link"/>
+			<xacro:insert_block name="joint_pose"/>
+			<axis xyz="0 1 0" rpy="0 0 0" />
+		</joint>
+		<transmission name="${wheel_prefix}_wheel_trans" type="SimpleTransmission">
+			<type>transmission_interface/SimpleTransmission</type>
+			<actuator name="${wheel_prefix}_wheel_motor">
+				<mechanicalReduction>1</mechanicalReduction>
+			</actuator>
+			<joint name="${wheel_prefix}_wheel">
+				<hardwareInterface>hardware_interface/VelocityJointInterface</hardwareInterface>
+			</joint>
+		</transmission>
+	</xacro:macro>
 </robot>
